File: thermocouple/Power.kicad_sch (KiCad schematic)
At the start: 19 parts, among them IC301 nPM1300-QEXX, X301 Charge, X302 Battery

Commit message: CI/CD improvements, fixing broken PMIC-INT
- Update CI/CD to the latest version
- Move PMIC-INT to port 0 to make it usable

Signed-off-by: Daniel Kampert <DanielKampert@kampis-elektroecke.de>
Parts:
- C301: footprint Resistor_SMD:R_0805_2012Metric -> Capacitor_SMD:C_0805_2012Metric; symbol Device:C_Small -> partdb:08053G105MAT2A; Category (none) -> Kondensator/MLCC; MPN (none) -> 08053G105MAT2A; Manufacturer (none) -> KYOCERA AVX; Manufacturing Status (none) -> Active; Mass (none) -> 0.006 g; Mouser SPN (none) -> 581-08053G105MAT2A; Part-DB Footprint (none) -> 0805; Part-DB ID (none) -> 349; Part-DB URL (none) -> https://inventory.lan/de/part/349/info; Stock (none) -> 0; manf# 08053C105K4Z2A -> 08053G105MAT2A; mouser# 581-08053C105K4Z2A -> 581-08053G105MAT2A
- C302: footprint Resistor_SMD:R_0805_2012Metric -> Capacitor_SMD:C_0805_2012Metric; symbol Device:C_Small -> partdb:08055C104K4Z4A; Category (none) -> Kondensator/MLCC; MPN (none) -> 08055C104K4Z4A; Manufacturer (none) -> KYOCERA AVX; Manufacturing Status (none) -> Active; Mass (none) -> 0.006 g; Mouser SPN (none) -> 581-08055C104K4Z4A; Part-DB Footprint (none) -> 0805; Part-DB ID (none) -> 109; Part-DB URL (none) -> https://inventory.lan/de/part/109/info; Stock (none) -> 6; Storage Location (none) -> Sortierregal; manf# 08053F104K4T2A -> 08055C104K4Z4A; mouser# 581-08053F104K4T2A -> 581-08055C104K4Z4A
- C303: footprint Resistor_SMD:R_0805_2012Metric -> Capacitor_SMD:C_0805_2012Metric; symbol Device:C_Small -> partdb:MCJCT21GCB7225MTPA1J; Category (none) -> Kondensator/MLCC; MPN (none) -> MCJCT21GCB7225MTPA1J; Manufacturer (none) -> TAIYO YUDEN; Manufacturing Status (none) -> Active; Mouser SPN (none) -> 963-T21GCB7225MTPA1J; Part-DB Footprint (none) -> 0805; Part-DB ID (none) -> 328; Part-DB URL (none) -> https://inventory.lan/de/part/328/info; Stock (none) -> 0; manf KYOCERA AVX -> TAIYO YUDEN; manf# 08052U220JAT2A -> MCJCT21GCB7225MTPA1J; mouser# 581-08052U220JAT2A -> 963-T21GCB7225MTPA1J
- C304, C305, C306, C307: footprint Resistor_SMD:R_0805_2012Metric -> Capacitor_SMD:C_0805_2012Metric; symbol Device:C_Small -> partdb:0805X7R106KT1AT; Category (none) -> Kondensator/MLCC; MPN (none) -> 0805X7R106KT1AT; Manufacturer (none) -> KYOCERA AVX; Manufacturing Status (none) -> Active; Mouser SPN (none) -> 581-0805X7R106KT1AT; Part-DB Footprint (none) -> 0805; Part-DB ID (none) -> 331; Part-DB URL (none) -> https://inventory.lan/de/part/331/info; Stock (none) -> 0; manf# KGM21AR71C106MU -> 0805X7R106KT1AT; mouser# 581-KGM21AR71C106MU -> 581-0805X7R106KT1AT
- L301: footprint Resistor_SMD:R_0805_2012Metric -> Inductor_SMD_Kampi:L_0806_2016; manf KYOCERA AVX -> ABRACON; manf# 08052U220JAT2A -> ASMPH-0806-2R2M-T; mouser# 581-08052U220JAT2A -> 815-ASMPH-0806-2R2M-T
- X302: manf (none) -> JST; manf# (none) -> S2B-PH-Sm4-TB
Other:
- moved on the sheet: C301, C302, C303, C304, C306, C307, TP303

Commit message: Reduce the brightnes of the status LED, use VSys for the LEDs
Parts:
- R401: value 590R -> 4k7; manf# CR0805-FX-5900ELF -> CR0805-JW-472ELF; mouser# 652-CR0805-FX-5900ELF -> 652-CR0805JW-472ELF
- R402: value 430R -> 10k; manf# CR0805-FX-4300ELF -> CR0805-FX-1002ELF; mouser# 652-CR0805-FX-4300ELF -> 652-CR0805FX-1002ELF
- R403: value 430R -> 3k3; manf# CR0805-FX-4300ELF -> CR0805-JW-332ELF; mouser# 652-CR0805-FX-4300ELF -> 652-CR0805-JW-332ELF
- X302: footprint Connector_JST:JST_PH_S2B-PH-SM4-TB_1x02-1MP_P2.00mm_Horizontal -> Connector_JST:JST_PH_B2B-PH-SM4-TB_1x02-1MP_P2.00mm_Vertical
Connections:
- net VSYS: now also D401.1 (A)
- net at C301.1, IC301.21 (V_{BUS}), X301.A4 (VBUS)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: no longer D401.1 (A)
Changed lines of the file:
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@@
 	)
 	(junction
-		(at 151.13 101.6)
-		(diameter 0)
-		(color 0 0 0 0)
-	)
-	(junction
 		(at 281.94 144.78)
 		(diameter 0)
@@
 	(wire
 		(pts
-			(xy 151.13 101.6) (xy 181.61 101.6)
-		)
-		(stroke
-			(width 0)
-			(type default)
-		)
-	)
-	(wire
-		(pts
 			(xy 274.32 74.93) (xy 287.02 74.93)
 		)
@@
 	(wire
 		(pts
-			(xy 213.36 83.82) (xy 219.71 83.82)
+			(xy 151.13 99.06) (xy 151.13 110.49)
 		)
 		(stroke
@@
 	(wire
 		(pts
-			(xy 125.73 101.6) (xy 151.13 101.6)
+			(xy 213.36 83.82) (xy 219.71 83.82)
 		)
 		(stroke
@@
 	(wire
 		(pts
-			(xy 151.13 101.6) (xy 151.13 110.49)
+			(xy 125.73 101.6) (xy 181.61 101.6)
 		)
 		(stroke
@@
 	)
 	(label "VSYS"
+		(at 151.13 99.06 90)
+		(effects
+			(font
+				(size 1.27 1.27)
+			)
+			(justify left bottom)
+		)
+	)
+	(label "VSYS"
 		(at 302.26 74.93 0)
 		(effects
@@
 			)
 		)
-		(property "Config" ""
-			(at 181.61 106.68 0)
-			(hide yes)
-			(show_name no)
-			(do_not_autoplace no)
-			(effects
-				(font
-					(size 1.27 1.27)
-				)
-			)
-		)
 		(property "Part-DB URL" "https://inventory.lan/de/part/349/info"
 			(at 181.61 106.68 0)
@@
 			)
 		)
-		(property "Config" ""
-			(at 281.94 149.86 0)
-			(hide yes)
-			(show_name no)
-			(do_not_autoplace no)
-			(effects
-				(font
-					(size 1.27 1.27)
-				)
-			)
-		)
 		(property "Part-DB URL" "https://inventory.lan/de/part/331/info"
 			(at 281.94 149.86 0)
@@
 			)
 		)
-		(property "Value" "590R"
+		(property "Value" "4k7"
 			(at 179.07 138.43 90)
 			(show_name no)
@@
 			)
 		)
-		(property "manf#" "CR0805-FX-5900ELF"
+		(property "manf#" "CR0805-JW-472ELF"
 			(at 179.07 142.24 0)
 			(hide yes)
@@
 			)
 		)
-		(property "mouser#" "652-CR0805-FX-5900ELF"
+		(property "mouser#" "652-CR0805JW-472ELF"
 			(at 179.07 142.24 0)
 			(hide yes)
@@
 			)
 		)
-		(property "Config" ""
-			(at 287.02 80.01 0)
-			(hide yes)
-			(show_name no)
-			(do_not_autoplace no)
-			(effects
-				(font
-					(size 1.27 1.27)
-				)
-			)
-		)
 		(property "Part-DB URL" "https://inventory.lan/de/part/331/info"
 			(at 287.02 80.01 0)
@@
 			)
 		)
-		(property "Config" ""
-			(at 271.78 149.86 0)
-			(hide yes)
-			(show_name no)
-			(do_not_autoplace no)
-			(effects
-				(font
-					(size 1.27 1.27)
-				)
-			)
-		)
 		(pin "1"
 		)
@@
 			)
 		)
-		(property "Footprint" "Connector_JST:JST_PH_S2B-PH-SM4-TB_1x02-1MP_P2.00mm_Horizontal"
+		(property "Footprint" "Connector_JST:JST_PH_B2B-PH-SM4-TB_1x02-1MP_P2.00mm_Vertical"
 			(at 248.92 82.55 0)
 			(hide yes)
@@
 			)
 		)
+		(property "mouser#" ""
+			(at 248.92 82.55 0)
+			(hide yes)
+			(show_name no)
+			(do_not_autoplace no)
+			(effects
+				(font
+					(size 1.27 1.27)
+				)
+			)
+		)
 		(pin "1"
 		)
@@
 			)
 		)
-		(property "Config" ""
-			(at 274.32 80.01 0)
-			(hide yes)
-			(show_name no)
-			(do_not_autoplace no)
-			(effects
-				(font
-					(size 1.27 1.27)
-				)
-			)
-		)
 		(property "Part-DB URL" "https://inventory.lan/de/part/331/info"
 			(at 274.32 80.01 0)
@@
 			)
 		)
-		(property "Value" "430R"
+		(property "Value" "3k3"
 			(at 163.83 133.35 90)
 			(show_name no)
@@
 			)
 		)
-		(property "manf#" "CR0805-FX-4300ELF"
+		(property "manf#" "CR0805-JW-332ELF"
 			(at 163.83 137.16 0)
 			(hide yes)
@@
 			)
 		)
-		(property "mouser#" "652-CR0805-FX-4300ELF"
+		(property "mouser#" "652-CR0805-JW-332ELF"
 			(at 163.83 137.16 0)
 			(hide yes)
@@
 			)
 		)
-		(property "Config" ""
-			(at 229.87 87.63 0)
-			(hide yes)
-			(show_name no)
-			(do_not_autoplace no)
-			(effects
-				(font
-					(size 1.27 1.27)
-				)
-			)
-		)
 		(property "Part-DB URL" "https://inventory.lan/de/part/328/info"
 			(at 229.87 87.63 0)
@@
 			)
 		)
-		(property "Value" "430R"
+		(property "Value" "10k"
 			(at 171.45 135.89 90)
 			(show_name no)
@@
 			)
 		)
-		(property "manf#" "CR0805-FX-4300ELF"
+		(property "manf#" "CR0805-FX-1002ELF"
 			(at 171.45 139.7 0)
 			(hide yes)
@@
 			)
 		)
-		(property "mouser#" "652-CR0805-FX-4300ELF"
+		(property "mouser#" "652-CR0805FX-1002ELF"
 			(at 171.45 139.7 0)
 			(hide yes)
@@
 			)
 		)
-		(property "Config" ""
-			(at 205.74 88.9 0)
-			(hide yes)
-			(show_name no)
-			(do_not_autoplace no)
-			(effects
-				(font
-					(size 1.27 1.27)
-				)
-			)
-		)
 		(property "Part-DB URL" "https://inventory.lan/de/part/109/info"
 			(at 205.74 88.9 0)
@@
 			)
 		)
-		(property "Config" ""
-			(at 300.99 80.01 0)
-			(hide yes)
-			(show_name no)
-			(do_not_autoplace no)
-			(effects
-				(font
-					(size 1.27 1.27)
-				)
-			)
-		)
 		(property "Part-DB URL" "https://inventory.lan/de/part/331/info"
 			(at 300.99 80.01 0)
@@
 			(at 110.49 116.84 0)
 			(hide yes)
-			(show_name no)
-			(do_not_autoplace no)
-			(effects
-				(font
-					(size 1.27 1.27)
-				)
-			)
-		)
-		(property "Config" ""
-			(at 110.49 116.84 0)
-			(hide yes)

Commit message: Change thermocouple connector to a different type
Parts:
- D401: symbol Device:LED_ARGB -> partdb:CLV1H-FKB-CM1R1H1BB23C4S3; Category (none) -> Diode/LED/RGB; MPN (none) -> CLV1H-FKB-CM1R1H1BB23C4S3; Manufacturer (none) -> Cree LED; Manufacturing Status (none) -> Active; Mouser SPN (none) -> 941-CLV1HBC1H1B3C4S3; Part-DB Footprint (none) -> PLCC4 3.2x2.8mm; Part-DB ID (none) -> 375; Part-DB URL (none) -> https://inventory.lan/de/part/375/info; Stock (none) -> 0
- X301: symbol Connector:USB_C_Receptacle_USB2.0_14P -> partdb:USB4110-GF-A; Category (none) -> Steckverbinder/USB; MPN (none) -> USB4110-GF-A; Manufacturer (none) -> GCT; Manufacturing Status (none) -> Active; Mass (none) -> 0.644 g; Mouser SPN (none) -> 640-USB4110-GF-A; Part-DB Footprint (none) -> USB4110; Part-DB ID (none) -> 369; Part-DB URL (none) -> https://inventory.lan/de/part/369/info; Stock (none) -> 0
- X302: footprint Connector_JST:JST_PH_B2B-PH-SM4-TB_1x02-1MP_P2.00mm_Vertical -> Connector_JST:JST_PH_S2B-PH-SM4-TB_1x02-1MP_P2.00mm_Horizontal
Connections:
- no-connect marks 17 -> 19
